Commit message: Created a launch file.
It starts the launch from qube_driver, rviz node, and robot_state_publisher node. It should be updated to include parameters which can be set when launching in the terminal.

Added world link in controlled_qube.urdf.xacro to actually display the robot defined in the macro.

File: qube_bringup/urdf/controlled_qube.urdf.xacro (robot description, xacro)
@@ -1,4 +1,4 @@
 <?xml version="1.0"?>
-<robot name="qube" xmlns:xacro="http://ros.org/wiki/xacro">
+<robot name="quanser_qube" xmlns:xacro="http://ros.org/wiki/xacro">
   <xacro:arg name="baud_rate" default="115200"/>
   <xacro:arg name="device" default="/dev/ttyUSB0"/> <!-- Double check what the default for device should be -->
@@ -6,4 +6,11 @@
   <xacro:include filename="$(find qube_description)/urdf/qube.macro.xacro" />
   <xacro:include filename="$(find qube_driver)/ros2_control/qube_driver.ros2_control.xacro"/>
+  <link name="world"/>
+  <xacro:qube prefix="" parent="world" />
+  <joint name="world_to_base_joint" type="fixed">
+    <parent link="world"/>
+    <child link="base_link"/> <!-- Adjust this name if your qube base link has a different name -->
+    <origin xyz="0 0 0" rpy="0 0 0"/>
+  </joint>
   <xacro:qube_driver_ros2_control
     name="qube_driver"

Commit message: removed two comments

File: qube_bringup/urdf/controlled_qube.urdf.xacro (robot description, xacro)
@@ -2,5 +2,5 @@
 <robot name="quanser_qube" xmlns:xacro="http://ros.org/wiki/xacro">
   <xacro:arg name="baud_rate" default="115200"/>
-  <xacro:arg name="device" default="/dev/ttyUSB0"/> <!-- Double check what the default for device should be -->
+  <xacro:arg name="device" default="/dev/ttyUSB0"/>
   <xacro:arg name="simulation" default="false"/>
   <xacro:include filename="$(find qube_description)/urdf/qube.macro.xacro" />
@@ -10,5 +10,5 @@
   <joint name="world_to_base_joint" type="fixed">
     <parent link="world"/>
-    <child link="base_link"/> <!-- Adjust this name if your qube base link has a different name -->
+    <child link="base_link"/>
     <origin xyz="0 0 0" rpy="0 0 0"/>
   </joint>
