Commit message: Added the new shapes (indicator and disc). The colors red and white are now defined too.
Made the joint connections from base_link (box) to the disc and the other joint connection from disc to indicator.

File: qube_description/qube.macro.xacro (robot description, xacro)
@@ -1,16 +1,73 @@
 <?xml version="1.0"?>
-<robot xmlns:xacro="http://www.ros.org/wiki/xacro" >
-  <! variabel definisjoner -->
+<robot xmlns:xacro="http://www.ros.org/wiki/xacro">
+  <!-- variabel definisjoner -->
   <xacro:property name = "qubeWidth" value = "0.5"/>
   <xacro:property name="qubeLength" value="0.5"/>
   <xacro:property name="qubeHeight" value="0.5"/>
-  <! farge variabler />
-  <xacro:property name="black" value="0 0 0 1"
-<xacro:macro name = "qube">
-  <link name = "black box">
-    <visual>
-      <geometry>
-        <box size = "${qubeWidth} ${qubeHeight} ${qubeLength}"/>
-      <geometry>
-      <material name="black"/>
-    </visual>
+  <xacro:property name="cylinderHeight" value="0.3"/>
+  <xacro:property name="cylinderRadius" value="0.5"/>
+  <xacro:property name="indicatorRadius" value="0.05"/>
+  <xacro:property name="indicatorLength" value="0.4"/>
+  <!-- farge variabler -->
+  <xacro:property name="black" value="0 0 0 1"/>
+  <xacro:property name="white" value="1 1 1 1"/>
+  <xacro:property name="red" value="1 0 0 1"/>
+  <xacro:macro name = "qube">
+    <link name = "base_link">
+      <visual>
+        <geometry>
+          <box size = "${qubeWidth} ${qubeLength} ${qubeHeight}"/>
+        </geometry>
+        <material name="black">
+          <color rgba = "${black}"/>
+        </material>
+      </visual>
+      <collision>
+        <geometry>
+          <box size="${qubeWidth} ${qubeLength} ${qubeHeight}"/>
+        </geometry>
+      </collision>
+    </link>
+    <link name="redDisc">
+      <visual>
+        <geometry>
+          <cylinder radius = "${cylinderRadius}" length = "${cylinderHeight}"/>
+        </geometry>
+        <material name="red">
+          <color rgba = "${red}"/>
+        </material>
+      </visual>
+      <collision>
+        <geometry>
+          <cylinder radius = "${cylinderRadius}" length = "${cylinderHeight}"/>
+        </geometry>
+      </collision>
+    </link>
+    <link name="whiteIndicator">
+      <visual>
+        <geometry>
+          <cylinder radius="${indicatorRadius}" length="${indicatorLength}"/>
+        </geometry>
+        <material name="white">
+          <color rgba = "${white}"/>
+        </material>
+      </visual>
+      <collision>
+        <geometry>
+          <cylinder radius="${indicatorRadius}" length="${indicatorLength}"/>
+        </geometry>
+      </collision>
+    </link>
+    <joint name="qube_to_disc" type = "continuous">
+      <parent link="base_link"/>
+      <child link="redDisc"/>
+      <origin xyz="0 0 ${qubeHeight/2 + cylinderHeight/2}" rpy="0 0 0"/>
+      <axis xyz="0 0 1"/>
+    </joint>
+    <joint name="disc_to_indicator" type="fixed">
+      <parent link="redDisc"/>
+      <child link="whiteIndicator"/>
+      <origin xyz="${cylinderRadius/2} 0 0" rpy="${pi/2} 0 0"/>
+    </joint>
+  </xacro:macro>
+</robot>
