Commit message: Edited the launch file to take arguments for the urdf parameters.
Using Command get the arguments into the robot description xacro. Getting the error "Joint 'motor_joint' not found in URDF" when launching in terminal. Also getting "[spawner-2] [INFO] [1743256098.997335899] [spawner_velocity_controller]: waiting for service /controller_manager/list_controllers to become available...
"

File: qube_description/urdf/qube.macro.xacro (robot description, xacro)
@@ -13,5 +13,5 @@
   <xacro:property name="white" value="1 1 1 1"/>
   <xacro:property name="red" value="1 0 0 1"/>
-  <xacro:macro name = "qube">
+  <xacro:macro name = "qube" params="prefix parent">
     <link name = "base_link">
       <visual>

Commit message: Defined the colors globally in the macro.xacro file, some parameters regarding the cylinder and the placement. Finished the urdf.xacro file too and started on the view_model.launch.py file

File: qube_description/urdf/qube.macro.xacro (robot description, xacro)
@@ -2,23 +2,30 @@
 <robot xmlns:xacro="http://www.ros.org/wiki/xacro">
   <!-- variabel definisjoner -->
-  <xacro:property name = "qubeWidth" value = "0.5"/>
+  <xacro:property name="qubeWidth" value="0.5"/>
   <xacro:property name="qubeLength" value="0.5"/>
   <xacro:property name="qubeHeight" value="0.5"/>
-  <xacro:property name="cylinderHeight" value="0.3"/>
-  <xacro:property name="cylinderRadius" value="0.5"/>
-  <xacro:property name="indicatorRadius" value="0.05"/>
-  <xacro:property name="indicatorLength" value="0.4"/>
+  <xacro:property name="cylinderHeight" value="0.1"/>
+  <xacro:property name="cylinderRadius" value="0.2"/>
+  <xacro:property name="indicatorRadius" value="0.02"/>
+  <xacro:property name="indicatorLength" value="0.15"/>
+  <xacro:property name="pi" value="3.1415926535897931"/>
   <!-- farge variabler -->
-  <xacro:property name="black" value="0 0 0 1"/>
-  <xacro:property name="white" value="1 1 1 1"/>
-  <xacro:property name="red" value="1 0 0 1"/>
+  <material name="black">
+    <color rgba="0 0 0 1"/>
+  </material>
+  <material name="red">
+    <color rgba="1 0 0 1"/>
+  </material>
+  <material name="white">
+    <color rgba="1 1 1 1"/>
+  </material>
   <xacro:macro name = "qube">
     <link name = "base_link">
       <visual>
         <geometry>
-          <box size = "${qubeWidth} ${qubeLength} ${qubeHeight}"/>
+          <box size ="${qubeWidth} ${qubeLength} ${qubeHeight}"/>
         </geometry>
         <material name="black">
-          <color rgba = "${black}"/>
+          <color rgba="${black}"/>
         </material>
       </visual>
@@ -32,13 +39,13 @@
       <visual>
         <geometry>
-          <cylinder radius = "${cylinderRadius}" length = "${cylinderHeight}"/>
+          <cylinder radius="${cylinderRadius}" length="${cylinderHeight}"/>
         </geometry>
         <material name="red">
-          <color rgba = "${red}"/>
+          <color rgba="${red}"/>
         </material>
       </visual>
       <collision>
         <geometry>
-          <cylinder radius = "${cylinderRadius}" length = "${cylinderHeight}"/>
+          <cylinder radius="${cylinderRadius}" length="${cylinderHeight}"/>
         </geometry>
       </collision>
@@ -50,5 +57,5 @@
         </geometry>
         <material name="white">
-          <color rgba = "${white}"/>
+          <color rgba="${white}"/>
         </material>
       </visual>
@@ -59,5 +66,5 @@
       </collision>
     </link>
-    <joint name="qube_to_disc" type = "continuous">
+    <joint name="qube_to_disc" type="continuous">
       <parent link="base_link"/>
       <child link="redDisc"/>
@@ -68,5 +75,5 @@
       <parent link="redDisc"/>
       <child link="whiteIndicator"/>
-      <origin xyz="${cylinderRadius/2} 0 0" rpy="${pi/2} 0 0"/>
+      <origin xyz="${cylinderRadius*0.7} 0 ${cylinderHeight/2}" rpy="${pi/2} 0 0"/>
     </joint>
   </xacro:macro>

Commit message: Change joint name of the red disk in qube macro to match the one in qube_driver, namely "motor_joint"

File: qube_description/urdf/qube.macro.xacro (robot description, xacro)
@@ -9,5 +9,5 @@
   <xacro:property name="indicatorRadius" value="0.02"/>
   <xacro:property name="indicatorLength" value="0.15"/>
-  <xacro:property name="pi" value="3.1415926535897931"/>
+<!--  <xacro:property name="pi" value="3.1415926535897931"/>-->
   <!-- farge variabler -->
   <material name="black">
@@ -26,7 +26,5 @@
           <box size ="${qubeWidth} ${qubeLength} ${qubeHeight}"/>
         </geometry>
-        <material name="black">
-          <color rgba="${black}"/>
-        </material>
+        <material name="black"/>
       </visual>
       <collision>
@@ -41,7 +39,5 @@
           <cylinder radius="${cylinderRadius}" length="${cylinderHeight}"/>
         </geometry>
-        <material name="red">
-          <color rgba="${red}"/>
-        </material>
+        <material name="red"/>
       </visual>
       <collision>
@@ -56,7 +52,5 @@
           <cylinder radius="${indicatorRadius}" length="${indicatorLength}"/>
         </geometry>
-        <material name="white">
-          <color rgba="${white}"/>
-        </material>
+        <material name="white"/>
       </visual>
       <collision>
@@ -66,5 +60,5 @@
       </collision>
     </link>
-    <joint name="qube_to_disc" type="continuous">
+    <joint name="motor_joint" type="continuous">
       <parent link="base_link"/>
       <child link="redDisc"/>

Commit message: changed values for height etc

File: qube_description/urdf/qube.macro.xacro (robot description, xacro)
@@ -5,9 +5,9 @@
   <xacro:property name="qubeLength" value="0.5"/>
   <xacro:property name="qubeHeight" value="0.5"/>
-  <xacro:property name="cylinderHeight" value="0.1"/>
-  <xacro:property name="cylinderRadius" value="0.2"/>
-  <xacro:property name="indicatorRadius" value="0.02"/>
-  <xacro:property name="indicatorLength" value="0.15"/>
-  <xacro:property name="pi" value="3.1415926535897931"/>
+  <xacro:property name="cylinderHeight" value="0.05"/>
+  <xacro:property name="cylinderRadius" value="0.1"/>
+  <xacro:property name="indicatorRadius" value="0.005"/>
+  <xacro:property name="indicatorLength" value="0.2"/>
+  <!-- <xacro:property name="pi" value="3.1415926535897931"/> -->
   <!-- farge variabler -->
   <material name="black">
@@ -75,5 +75,5 @@
       <parent link="redDisc"/>
       <child link="whiteIndicator"/>
-      <origin xyz="${cylinderRadius*0.7} 0 ${cylinderHeight/2}" rpy="${pi/2} 0 0"/>
+      <origin xyz="0 0 ${cylinderHeight/2}" rpy="${pi/3} 0 0"/>
     </joint>
   </xacro:macro>

Commit message: Added the second indicator and all the properties for it with the joint for it being connected to the "redDisk"

File: qube_description/urdf/qube.macro.xacro (robot description, xacro)
@@ -5,9 +5,13 @@
   <xacro:property name="qubeLength" value="0.5"/>
   <xacro:property name="qubeHeight" value="0.5"/>
-  <xacro:property name="cylinderHeight" value="0.1"/>
-  <xacro:property name="cylinderRadius" value="0.2"/>
-  <xacro:property name="indicatorRadius" value="0.02"/>
-  <xacro:property name="indicatorLength" value="0.15"/>
-<!--  <xacro:property name="pi" value="3.1415926535897931"/>-->
+  <xacro:property name="cylinderHeight" value="0.04"/>
+  <xacro:property name="cylinderRadius" value="0.07"/>
+  <xacro:property name="indicatorWidth" value="0.005"/>
+  <xacro:property name="indicatorLength" value="0.14"/>
+  <xacro:property name="indicatorHeight" value="0.001"/>
+  <xacro:property name="sIndicatorL" value="0.07"/>
+  <xacro:property name="sIndicatorW" value="0.005"/>
+  <xacro:property name="sIndicatorH" value="0.001"/>
+  <xacro:property name="pi" value="3.1415926535897931"/>
   <!-- farge variabler -->
   <material name="black">
@@ -20,5 +24,5 @@
     <color rgba="1 1 1 1"/>
   </material>
-  <xacro:macro name = "qube" params="prefix parent">
+  <xacro:macro name="qube">
     <link name = "base_link">
       <visual>
@@ -50,5 +54,5 @@
       <visual>
         <geometry>
-          <cylinder radius="${indicatorRadius}" length="${indicatorLength}"/>
+          <box size="${indicatorLength} ${indicatorHeight} ${indicatorWidth}"/>
         </geometry>
         <material name="white"/>
@@ -56,5 +60,18 @@
       <collision>
         <geometry>
-          <cylinder radius="${indicatorRadius}" length="${indicatorLength}"/>
+          <box size="${indicatorLength}  ${indicatorHeight} ${indicatorWidth}"/>
+        </geometry>
+      </collision>
+    </link>
+    <link name="sIndicator">
+      <visual>
+        <geometry>
+          <box size="${sIndicatorL} ${sIndicatorH} ${sIndicatorW}"/>
+        </geometry>
+        <material name="white"/>
+      </visual>
+      <collision>
+        <geometry>
+          <box size="${sIndicatorL} ${sIndicatorH} ${sIndicatorW}"/>
         </geometry>
       </collision>
@@ -69,5 +86,10 @@
       <parent link="redDisc"/>
       <child link="whiteIndicator"/>
-      <origin xyz="${cylinderRadius*0.7} 0 ${cylinderHeight/2}" rpy="${pi/2} 0 0"/>
+      <origin xyz="0 0 ${cylinderHeight/2}" rpy="${pi/2} 0 0"/>
+    </joint>
+    <joint name="sIndicator2disc" type="fixed">
+      <parent link="redDisc"/>
+      <child link="sIndicator"/>
+      <origin xyz="0 0 ${cylinderHeight/2}" rpy="0 0 0"/>
     </joint>
   </xacro:macro>

Commit message: added second indicator (sIndicator) and the joint for it to be connected with the red disc (redDisc)

File: qube_description/urdf/qube.macro.xacro (robot description, xacro)
@@ -13,5 +13,4 @@
   <xacro:property name="sIndicatorW" value="0.005"/>
   <xacro:property name="sIndicatorH" value="0.001"/>
-  <xacro:property name="pi" value="3.1415926535897931"/>
   <!-- farge variabler -->
   <material name="black">
@@ -91,5 +90,5 @@
       <parent link="redDisc"/>
       <child link="sIndicator"/>
-      <origin xyz="0 0 ${cylinderHeight/2}" rpy="0 0 0"/>
+       <origin xyz="${cylinderRadius/2} 0 ${cylinderHeight/2}" rpy="0 0 0"/>
     </joint>
   </xacro:macro>

Commit message: fixed tuple error and the RViz problem where the robot did not show

File: qube_description/urdf/qube.macro.xacro (robot description, xacro)
@@ -5,9 +5,13 @@
   <xacro:property name="qubeLength" value="0.5"/>
   <xacro:property name="qubeHeight" value="0.5"/>
-  <xacro:property name="cylinderHeight" value="0.1"/>
-  <xacro:property name="cylinderRadius" value="0.2"/>
-  <xacro:property name="indicatorRadius" value="0.02"/>
-  <xacro:property name="indicatorLength" value="0.15"/>
-<!--  <xacro:property name="pi" value="3.1415926535897931"/>-->
+  <xacro:property name="cylinderHeight" value="0.04"/>
+  <xacro:property name="cylinderRadius" value="0.07"/>
+  <xacro:property name="indicatorWidth" value="0.005"/>
+  <xacro:property name="indicatorLength" value="0.14"/>
+  <xacro:property name="indicatorHeight" value="0.001"/>
+  <xacro:property name="sIndicatorL" value="0.07"/>
+  <xacro:property name="sIndicatorW" value="0.005"/>
+  <xacro:property name="sIndicatorH" value="0.001"/>
+  <!--  <xacro:property name="pi" value="3.1415926535897931"/>-->
   <!-- farge variabler -->
   <material name="black">
@@ -50,5 +54,5 @@
       <visual>
         <geometry>
-          <cylinder radius="${indicatorRadius}" length="${indicatorLength}"/>
+          <box size="${indicatorLength} ${indicatorHeight} ${indicatorWidth}"/>
         </geometry>
         <material name="white"/>
@@ -56,5 +60,18 @@
       <collision>
         <geometry>
-          <cylinder radius="${indicatorRadius}" length="${indicatorLength}"/>
+          <box size="${indicatorLength}  ${indicatorHeight} ${indicatorWidth}"/>
+        </geometry>
+      </collision>
+    </link>
+    <link name="sIndicator">
+      <visual>
+        <geometry>
+          <box size="${sIndicatorL} ${sIndicatorH} ${sIndicatorW}"/>
+        </geometry>
+        <material name="white"/>
+      </visual>
+      <collision>
+        <geometry>
+          <box size="${sIndicatorL} ${sIndicatorH} ${sIndicatorW}"/>
         </geometry>
       </collision>
@@ -69,5 +86,10 @@
       <parent link="redDisc"/>
       <child link="whiteIndicator"/>
-      <origin xyz="${cylinderRadius*0.7} 0 ${cylinderHeight/2}" rpy="${pi/2} 0 0"/>
+      <origin xyz="0 0 ${cylinderHeight/2}" rpy="${pi/2} 0 0"/>
+    </joint>
+    <joint name="sIndicator2disc" type="fixed">
+      <parent link="redDisc"/>
+      <child link="sIndicator"/>
+       <origin xyz="${cylinderRadius/2} 0 ${cylinderHeight/2}" rpy="0 0 0"/>
     </joint>
   </xacro:macro>

Commit message: Fixed the measurements for the redDisc and the whiteIndicator and sIndicator so they represent the quanser qube more correctly

File: qube_description/urdf/qube.macro.xacro (robot description, xacro)
@@ -6,12 +6,12 @@
   <xacro:property name="qubeHeight" value="0.5"/>
   <xacro:property name="cylinderHeight" value="0.04"/>
-  <xacro:property name="cylinderRadius" value="0.07"/>
+  <xacro:property name="cylinderRadius" value="0.11"/>
   <xacro:property name="indicatorWidth" value="0.005"/>
-  <xacro:property name="indicatorLength" value="0.14"/>
+  <xacro:property name="indicatorLength" value="0.22"/>
   <xacro:property name="indicatorHeight" value="0.001"/>
-  <xacro:property name="sIndicatorL" value="0.07"/>
+  <xacro:property name="sIndicatorL" value="0.11"/>
   <xacro:property name="sIndicatorW" value="0.005"/>
   <xacro:property name="sIndicatorH" value="0.001"/>
-  <!--  <xacro:property name="pi" value="3.1415926535897931"/>-->
+  <!-- <xacro:property name="pi" value="3.1415926535897931"/> -->
   <!-- farge variabler -->
   <material name="black">
@@ -40,6 +40,9 @@
     <link name="redDisc">
       <visual>
+        <origin xyz="0 0 0" rpy="0.001 0.001 0"/>
         <geometry>
-          <cylinder radius="${cylinderRadius}" length="${cylinderHeight}"/>
+          <cylinder radius="${cylinderRadius}" length="${cylinderHeight}">
+            <resolution>50</resolution>
+          </cylinder>
         </geometry>
         <material name="red"/>
@@ -66,4 +69,5 @@
     <link name="sIndicator">
       <visual>
+        <origin xyz="${sIndicatorL/2} 0 0"/>
         <geometry>
           <box size="${sIndicatorL} ${sIndicatorH} ${sIndicatorW}"/>
@@ -72,4 +76,5 @@
       </visual>
       <collision>
+        <origin xyz="${sIndicatorL/2} 0 0"/>
         <geometry>
           <box size="${sIndicatorL} ${sIndicatorH} ${sIndicatorW}"/>
@@ -91,5 +96,5 @@
       <parent link="redDisc"/>
       <child link="sIndicator"/>
-       <origin xyz="${cylinderRadius/2} 0 ${cylinderHeight/2}" rpy="0 0 0"/>
+       <origin xyz="0 0 ${cylinderHeight/2}" rpy="${pi/2} 0 ${pi/2}"/>
     </joint>
   </xacro:macro>

Commit message: its not working, I cant run the eike3 launch for qube_description (view_qube.launch.py), and the bringup.launch.py one doesnt work eitehr. we are not sure what the probelm is but its probably something with the launch file for qube_description.

File: qube_description/urdf/qube.macro.xacro (robot description, xacro)
@@ -43,5 +43,5 @@
         <geometry>
           <cylinder radius="${cylinderRadius}" length="${cylinderHeight}">
-            <resolution>50</resolution>
+            <!--<resolution>50</resolution>-->
           </cylinder>
         </geometry>
@@ -91,10 +91,10 @@
       <parent link="redDisc"/>
       <child link="whiteIndicator"/>
-      <origin xyz="0 0 ${cylinderHeight/2}" rpy="${pi/2} 0 0"/>
+      <origin xyz="0 0 ${cylinderHeight/2}" rpy="${3/2} 0 0"/>
     </joint>
     <joint name="sIndicator2disc" type="fixed">
       <parent link="redDisc"/>
       <child link="sIndicator"/>
-       <origin xyz="0 0 ${cylinderHeight/2}" rpy="${pi/2} 0 ${pi/2}"/>
+       <origin xyz="0 0 ${cylinderHeight/2}" rpy="${3/2} 0 ${3/2}"/>
     </joint>
   </xacro:macro>

File: qube_description/urdf/qube.urdf.xacro (robot description, xacro)
@@ -1,12 +1,11 @@
 <?xml version="1.0"?>
-<robot xmlns:xacro="http://www.ros.org/wiki/xacro" >
-	<xacro:include filename="$(find qube_description)/urdf/qube.macro.xacro" />
-  <link name="world">
-  </link>
-  <xacro:qube/>
-  <joint name="world_to_qube" type="fixed">
-    <origin xyz="0 0 0" rpy="0 0 0"/>
+<robot name="quanser_qube" xmlns:xacro="http://ros.org/wiki/xacro" >
+	<xacro:include filename="$(find qube_description)/urdf/qube.macro.xacro"/>
+  <link name="world"/>
+  <xacro:qube prefix="" parent="world"/>
+  <joint name="world_to_base_joint" type="fixed">
     <parent link="world"/>
     <child link="base_link"/>
+    <origin xyz="0 0 0" rpy="0 0 0"/>
   </joint>
 </robot>

Commit message: added macro.xacro from eike3

File: qube_description/urdf/qube.macro.xacro (robot description, xacro)
@@ -5,9 +5,13 @@
   <xacro:property name="qubeLength" value="0.5"/>
   <xacro:property name="qubeHeight" value="0.5"/>
-  <xacro:property name="cylinderHeight" value="0.1"/>
-  <xacro:property name="cylinderRadius" value="0.2"/>
-  <xacro:property name="indicatorRadius" value="0.02"/>
-  <xacro:property name="indicatorLength" value="0.15"/>
-<!--  <xacro:property name="pi" value="3.1415926535897931"/>-->
+  <xacro:property name="cylinderHeight" value="0.04"/>
+  <xacro:property name="cylinderRadius" value="0.11"/>
+  <xacro:property name="indicatorWidth" value="0.005"/>
+  <xacro:property name="indicatorLength" value="0.22"/>
+  <xacro:property name="indicatorHeight" value="0.001"/>
+  <xacro:property name="sIndicatorL" value="0.11"/>
+  <xacro:property name="sIndicatorW" value="0.005"/>
+  <xacro:property name="sIndicatorH" value="0.001"/>
+  <!-- <xacro:property name="pi" value="3.1415926535897931"/> -->
   <!-- farge variabler -->
   <material name="black">
@@ -36,6 +40,9 @@
     <link name="redDisc">
       <visual>
+        <origin xyz="0 0 0" rpy="0.001 0.001 0"/>
         <geometry>
-          <cylinder radius="${cylinderRadius}" length="${cylinderHeight}"/>
+          <cylinder radius="${cylinderRadius}" length="${cylinderHeight}">
+            <!--<resolution>50</resolution>-->
+          </cylinder>
         </geometry>
         <material name="red"/>
@@ -50,5 +57,5 @@
       <visual>
         <geometry>
-          <cylinder radius="${indicatorRadius}" length="${indicatorLength}"/>
+          <box size="${indicatorLength} ${indicatorHeight} ${indicatorWidth}"/>
         </geometry>
         <material name="white"/>
@@ -56,5 +63,20 @@
       <collision>
         <geometry>
-          <cylinder radius="${indicatorRadius}" length="${indicatorLength}"/>
+          <box size="${indicatorLength}  ${indicatorHeight} ${indicatorWidth}"/>
+        </geometry>
+      </collision>
+    </link>
+    <link name="sIndicator">
+      <visual>
+        <origin xyz="${sIndicatorL/2} 0 0"/>
+        <geometry>
+          <box size="${sIndicatorL} ${sIndicatorH} ${sIndicatorW}"/>
+        </geometry>
+        <material name="white"/>
+      </visual>
+      <collision>
+        <origin xyz="${sIndicatorL/2} 0 0"/>
+        <geometry>
+          <box size="${sIndicatorL} ${sIndicatorH} ${sIndicatorW}"/>
         </geometry>
       </collision>
@@ -69,5 +91,10 @@
       <parent link="redDisc"/>
       <child link="whiteIndicator"/>
-      <origin xyz="${cylinderRadius*0.7} 0 ${cylinderHeight/2}" rpy="${pi/2} 0 0"/>
+      <origin xyz="0 0 ${cylinderHeight/2}" rpy="${3/2} 0 0"/>
+    </joint>
+    <joint name="sIndicator2disc" type="fixed">
+      <parent link="redDisc"/>
+      <child link="sIndicator"/>
+       <origin xyz="0 0 ${cylinderHeight/2}" rpy="${3/2} 0 ${3/2}"/>
     </joint>
   </xacro:macro>

Commit message: The gray disc under the red one is now added with some joint adjustments so the new robot includes the gray disc. Also I did some adjustments to the setup.py file, added qube.rviz file, and some changes to the launch file, by doing these adjustments the qube_description is now able to launch using the view_qube.launch.py launch file

File: qube_description/urdf/qube.macro.xacro (robot description, xacro)
@@ -13,4 +13,6 @@
   <xacro:property name="sIndicatorW" value="0.005"/>
   <xacro:property name="sIndicatorH" value="0.001"/>
+  <xacro:property name="grayCylinderH" value="0.06"/>
+  <xacro:property name="grayCylinderR" value="0.05"/>
   <!-- <xacro:property name="pi" value="3.1415926535897931"/> -->
   <!-- farge variabler -->
@@ -23,4 +25,7 @@
   <material name="white">
     <color rgba="1 1 1 1"/>
+  </material>
+  <material name="gray">
+    <color rgba="0.5 0.5 0.5 1"/>
   </material>
   <xacro:macro name = "qube" params="prefix parent">
@@ -82,7 +87,22 @@
       </collision>
     </link>
+    <link name="grayDisc">
+      <visual>
+        <origin xyz="0 0 0"/>
+        <geometry>
+          <cylinder length="${grayCylinderH}" radius="${grayCylinderR}"/>
+        </geometry>
+        <material name="gray"/>
+      </visual>
+      <collision>
+        <origin xyz="0 0 0"/>
+        <geometry>
+          <cylinder length="${grayCylinderH}" radius="${grayCylinderR}"/>
+        </geometry>
+      </collision>
+    </link>
     <joint name="motor_joint" type="continuous">
       <parent link="base_link"/>
-      <child link="redDisc"/>
+      <child link="grayDisc"/>
       <origin xyz="0 0 ${qubeHeight/2 + cylinderHeight/2}" rpy="0 0 0"/>
       <axis xyz="0 0 1"/>
@@ -96,5 +116,10 @@
       <parent link="redDisc"/>
       <child link="sIndicator"/>
-       <origin xyz="0 0 ${cylinderHeight/2}" rpy="${3/2} 0 ${3/2}"/>
+      <origin xyz="0 0 ${cylinderHeight/2}" rpy="${3/2} 0 ${3/2}"/>
+    </joint>
+    <joint name="disc_to_disc" type="fixed">
+      <parent link="grayDisc"/>
+      <child link="redDisc"/>
+      <origin xyz="0 0 ${grayCylinderH/2}"/>
     </joint>
   </xacro:macro>

Commit message: Added the red line to the robot for better detail

File: qube_description/urdf/qube.macro.xacro (robot description, xacro)
@@ -15,4 +15,7 @@
   <xacro:property name="grayCylinderH" value="0.06"/>
   <xacro:property name="grayCylinderR" value="0.05"/>
+  <xacro:property name="redLineW" value="0.501"/>
+  <xacro:property name="redLineL" value="0.501"/>
+  <xacro:property name="redLineH" value="0.01"/>
   <!-- <xacro:property name="pi" value="3.1415926535897931"/> -->
   <!-- farge variabler -->
@@ -102,4 +105,19 @@
       </collision>
     </link>
+    <link name="redLine">
+      <visual>
+        <origin xyz="0 0 0"/>
+        <geometry>
+          <box size="${redLineW} ${redLineL} ${redLineH}"/>
+        </geometry>
+        <material name="red"/>
+      </visual>
+      <collision>
+        <origin xyz="0 0 0"/>
+        <geometry>
+          <box size="${redLineW} ${redLineL} ${redLineH}"/>
+        </geometry>
+      </collision>
+    </link>
     <joint name="motor_joint" type="continuous">
       <parent link="base_link"/>
@@ -123,4 +141,9 @@
       <origin xyz="0 0 ${grayCylinderH/2}"/>
     </joint>
+    <joint name="redLineToBox" type="fixed">
+      <parent link="base_link"/>
+      <child link="redLine"/>
+       <origin xyz="0 0 ${qubeHeight/2 - 0.01}"/>
+    </joint>
   </xacro:macro>
 </robot>
